Commit message: Removed hebi parameters from configs

File: hebi_a-2084-01-parallel-gripper_moveit_config/config/A-2084-01-parallel-gripper.ros2_control.xacro (robot description, xacro)
@@ -3,32 +3,8 @@
     <xacro:macro name="A-2084-01-parallel-gripper_ros2_control" params="name initial_positions_file">
         <xacro:property name="initial_positions" value="${load_yaml(initial_positions_file)['initial_positions']}"/>
-        <xacro:property name="home_position" value="${load_yaml(initial_positions_file)['home_position']}"/>
-        <xacro:property name="families" value="${load_yaml(initial_positions_file)['families']}"/>
-        <xacro:property name="names" value="${load_yaml(initial_positions_file)['names']}"/>
-        <xacro:property name="hrdf_pkg" value="${load_yaml(initial_positions_file)['hrdf_pkg']}"/>
-        <xacro:property name="hrdf_file" value="${load_yaml(initial_positions_file)['hrdf_file']}"/>
-        <xacro:property name="gains_pkg" value="${load_yaml(initial_positions_file)['gains_pkg']}"/>
-        <xacro:property name="gains_file" value="${load_yaml(initial_positions_file)['gains_file']}"/>
-        <xacro:property name="use_mock_hardware" value="${load_yaml(initial_positions_file)['use_mock_hardware']}"/>
-        <xacro:property name="use_gazebo" value="${load_yaml(initial_positions_file)['use_gazebo']}"/>
         <ros2_control name="${name}" type="system">
             <hardware>
-              <xacro:if value="${use_mock_hardware}">
+                <!-- By default, set up controllers for simulation. This won't work on real hardware -->
                 <plugin>mock_components/GenericSystem</plugin>
-              </xacro:if>
-              <xacro:if value="${use_gazebo}">
-                <plugin>gazebo_ros2_control/GazeboSystem</plugin>
-              </xacro:if>
-              <xacro:unless value="${use_mock_hardware or use_gazebo}">
-                <!-- Parameters to initialize the Components -->
-                <param name="families">${families}</param>
-                <param name="names">${names}</param>
-                <param name="hrdf_pkg">${hrdf_pkg}</param>
-                <param name="hrdf_file">${hrdf_file}</param>
-                <param name="gains_pkg">${gains_pkg}</param>
-                <param name="gains_file">${gains_file}</param>
-                <param name="home_position">${home_position}</param>
-                <plugin>hebi_hardware/HEBIHardwareInterface</plugin>
-              </xacro:unless>
             </hardware>
             <joint name="J1_base">

File: hebi_a-2084-01_moveit_config/config/A-2084-01.ros2_control.xacro (robot description, xacro)
@@ -3,32 +3,8 @@
     <xacro:macro name="A-2084-01_ros2_control" params="name initial_positions_file">
         <xacro:property name="initial_positions" value="${load_yaml(initial_positions_file)['initial_positions']}"/>
-        <xacro:property name="home_position" value="${load_yaml(initial_positions_file)['home_position']}"/>
-        <xacro:property name="families" value="${load_yaml(initial_positions_file)['families']}"/>
-        <xacro:property name="names" value="${load_yaml(initial_positions_file)['names']}"/>
-        <xacro:property name="hrdf_pkg" value="${load_yaml(initial_positions_file)['hrdf_pkg']}"/>
-        <xacro:property name="hrdf_file" value="${load_yaml(initial_positions_file)['hrdf_file']}"/>
-        <xacro:property name="gains_pkg" value="${load_yaml(initial_positions_file)['gains_pkg']}"/>
-        <xacro:property name="gains_file" value="${load_yaml(initial_positions_file)['gains_file']}"/>
-        <xacro:property name="use_mock_hardware" value="${load_yaml(initial_positions_file)['use_mock_hardware']}"/>
-        <xacro:property name="use_gazebo" value="${load_yaml(initial_positions_file)['use_gazebo']}"/>
         <ros2_control name="${name}" type="system">
             <hardware>
-              <xacro:if value="${use_mock_hardware}">
+                <!-- By default, set up controllers for simulation. This won't work on real hardware -->
                 <plugin>mock_components/GenericSystem</plugin>
-              </xacro:if>
-              <xacro:if value="${use_gazebo}">
-                <plugin>gazebo_ros2_control/GazeboSystem</plugin>
-              </xacro:if>
-              <xacro:unless value="${use_mock_hardware or use_gazebo}">
-                <!-- Parameters to initialize the Components -->
-                <param name="families">${families}</param>
-                <param name="names">${names}</param>
-                <param name="hrdf_pkg">${hrdf_pkg}</param>
-                <param name="hrdf_file">${hrdf_file}</param>
-                <param name="gains_pkg">${gains_pkg}</param>
-                <param name="gains_file">${gains_file}</param>
-                <param name="home_position">${home_position}</param>
-                <plugin>hebi_hardware/HEBIHardwareInterface</plugin>
-              </xacro:unless>
             </hardware>
             <joint name="J1_base">

File: hebi_a-2085-04-parallel-gripper_moveit_config/config/A-2085-04-parallel-gripper.ros2_control.xacro (robot description, xacro)
@@ -3,32 +3,8 @@
     <xacro:macro name="A-2085-04-parallel-gripper_ros2_control" params="name initial_positions_file">
         <xacro:property name="initial_positions" value="${load_yaml(initial_positions_file)['initial_positions']}"/>
-        <xacro:property name="home_position" value="${load_yaml(initial_positions_file)['home_position']}"/>
-        <xacro:property name="families" value="${load_yaml(initial_positions_file)['families']}"/>
-        <xacro:property name="names" value="${load_yaml(initial_positions_file)['names']}"/>
-        <xacro:property name="hrdf_pkg" value="${load_yaml(initial_positions_file)['hrdf_pkg']}"/>
-        <xacro:property name="hrdf_file" value="${load_yaml(initial_positions_file)['hrdf_file']}"/>
-        <xacro:property name="gains_pkg" value="${load_yaml(initial_positions_file)['gains_pkg']}"/>
-        <xacro:property name="gains_file" value="${load_yaml(initial_positions_file)['gains_file']}"/>
-        <xacro:property name="use_mock_hardware" value="${load_yaml(initial_positions_file)['use_mock_hardware']}"/>
-        <xacro:property name="use_gazebo" value="${load_yaml(initial_positions_file)['use_gazebo']}"/>
         <ros2_control name="${name}" type="system">
             <hardware>
-              <xacro:if value="${use_mock_hardware}">
+                <!-- By default, set up controllers for simulation. This won't work on real hardware -->
                 <plugin>mock_components/GenericSystem</plugin>
-              </xacro:if>
-              <xacro:if value="${use_gazebo}">
-                <plugin>gazebo_ros2_control/GazeboSystem</plugin>
-              </xacro:if>
-              <xacro:unless value="${use_mock_hardware or use_gazebo}">
-                <!-- Parameters to initialize the Components -->
-                <param name="families">${families}</param>
-                <param name="names">${names}</param>
-                <param name="hrdf_pkg">${hrdf_pkg}</param>
-                <param name="hrdf_file">${hrdf_file}</param>
-                <param name="gains_pkg">${gains_pkg}</param>
-                <param name="gains_file">${gains_file}</param>
-                <param name="home_position">${home_position}</param>
-                <plugin>hebi_hardware/HEBIHardwareInterface</plugin>
-              </xacro:unless>
             </hardware>
             <joint name="J1_base">

File: hebi_a-2085-04_moveit_config/config/A-2085-04.ros2_control.xacro (robot description, xacro)
@@ -3,32 +3,8 @@
     <xacro:macro name="A-2085-04_ros2_control" params="name initial_positions_file">
         <xacro:property name="initial_positions" value="${load_yaml(initial_positions_file)['initial_positions']}"/>
-        <xacro:property name="home_position" value="${load_yaml(initial_positions_file)['home_position']}"/>
-        <xacro:property name="families" value="${load_yaml(initial_positions_file)['families']}"/>
-        <xacro:property name="names" value="${load_yaml(initial_positions_file)['names']}"/>
-        <xacro:property name="hrdf_pkg" value="${load_yaml(initial_positions_file)['hrdf_pkg']}"/>
-        <xacro:property name="hrdf_file" value="${load_yaml(initial_positions_file)['hrdf_file']}"/>
-        <xacro:property name="gains_pkg" value="${load_yaml(initial_positions_file)['gains_pkg']}"/>
-        <xacro:property name="gains_file" value="${load_yaml(initial_positions_file)['gains_file']}"/>
-        <xacro:property name="use_mock_hardware" value="${load_yaml(initial_positions_file)['use_mock_hardware']}"/>
-        <xacro:property name="use_gazebo" value="${load_yaml(initial_positions_file)['use_gazebo']}"/>
         <ros2_control name="${name}" type="system">
             <hardware>
-              <xacro:if value="${use_mock_hardware}">
+                <!-- By default, set up controllers for simulation. This won't work on real hardware -->
                 <plugin>mock_components/GenericSystem</plugin>
-              </xacro:if>
-              <xacro:if value="${use_gazebo}">
-                <plugin>gazebo_ros2_control/GazeboSystem</plugin>
-              </xacro:if>
-              <xacro:unless value="${use_mock_hardware or use_gazebo}">
-                <!-- Parameters to initialize the Components -->
-                <param name="families">${families}</param>
-                <param name="names">${names}</param>
-                <param name="hrdf_pkg">${hrdf_pkg}</param>
-                <param name="hrdf_file">${hrdf_file}</param>
-                <param name="gains_pkg">${gains_pkg}</param>
-                <param name="gains_file">${gains_file}</param>
-                <param name="home_position">${home_position}</param>
-                <plugin>hebi_hardware/HEBIHardwareInterface</plugin>
-              </xacro:unless>
             </hardware>
             <joint name="J1_base">

File: hebi_a-2085-05-parallel-gripper_moveit_config/config/A-2085-05-parallel-gripper.ros2_control.xacro (robot description, xacro)
@@ -3,32 +3,8 @@
     <xacro:macro name="A-2085-05-parallel-gripper_ros2_control" params="name initial_positions_file">
         <xacro:property name="initial_positions" value="${load_yaml(initial_positions_file)['initial_positions']}"/>
-        <xacro:property name="home_position" value="${load_yaml(initial_positions_file)['home_position']}"/>
-        <xacro:property name="families" value="${load_yaml(initial_positions_file)['families']}"/>
-        <xacro:property name="names" value="${load_yaml(initial_positions_file)['names']}"/>
-        <xacro:property name="hrdf_pkg" value="${load_yaml(initial_positions_file)['hrdf_pkg']}"/>
-        <xacro:property name="hrdf_file" value="${load_yaml(initial_positions_file)['hrdf_file']}"/>
-        <xacro:property name="gains_pkg" value="${load_yaml(initial_positions_file)['gains_pkg']}"/>
-        <xacro:property name="gains_file" value="${load_yaml(initial_positions_file)['gains_file']}"/>
-        <xacro:property name="use_mock_hardware" value="${load_yaml(initial_positions_file)['use_mock_hardware']}"/>
-        <xacro:property name="use_gazebo" value="${load_yaml(initial_positions_file)['use_gazebo']}"/>
         <ros2_control name="${name}" type="system">
             <hardware>
-              <xacro:if value="${use_mock_hardware}">
+                <!-- By default, set up controllers for simulation. This won't work on real hardware -->
                 <plugin>mock_components/GenericSystem</plugin>
-              </xacro:if>
-              <xacro:if value="${use_gazebo}">
-                <plugin>gazebo_ros2_control/GazeboSystem</plugin>
-              </xacro:if>
-              <xacro:unless value="${use_mock_hardware or use_gazebo}">
-                <!-- Parameters to initialize the Components -->
-                <param name="families">${families}</param>
-                <param name="names">${names}</param>
-                <param name="hrdf_pkg">${hrdf_pkg}</param>
-                <param name="hrdf_file">${hrdf_file}</param>
-                <param name="gains_pkg">${gains_pkg}</param>
-                <param name="gains_file">${gains_file}</param>
-                <param name="home_position">${home_position}</param>
-                <plugin>hebi_hardware/HEBIHardwareInterface</plugin>
-              </xacro:unless>
             </hardware>
             <joint name="J1_base">

File: hebi_a-2085-05_moveit_config/config/A-2085-05.ros2_control.xacro (robot description, xacro)
@@ -3,32 +3,8 @@
     <xacro:macro name="A-2085-05_ros2_control" params="name initial_positions_file">
         <xacro:property name="initial_positions" value="${load_yaml(initial_positions_file)['initial_positions']}"/>
-        <xacro:property name="home_position" value="${load_yaml(initial_positions_file)['home_position']}"/>
-        <xacro:property name="families" value="${load_yaml(initial_positions_file)['families']}"/>
-        <xacro:property name="names" value="${load_yaml(initial_positions_file)['names']}"/>
-        <xacro:property name="hrdf_pkg" value="${load_yaml(initial_positions_file)['hrdf_pkg']}"/>
-        <xacro:property name="hrdf_file" value="${load_yaml(initial_positions_file)['hrdf_file']}"/>
-        <xacro:property name="gains_pkg" value="${load_yaml(initial_positions_file)['gains_pkg']}"/>
-        <xacro:property name="gains_file" value="${load_yaml(initial_positions_file)['gains_file']}"/>
-        <xacro:property name="use_mock_hardware" value="${load_yaml(initial_positions_file)['use_mock_hardware']}"/>
-        <xacro:property name="use_gazebo" value="${load_yaml(initial_positions_file)['use_gazebo']}"/>
         <ros2_control name="${name}" type="system">
             <hardware>
-              <xacro:if value="${use_mock_hardware}">
+                <!-- By default, set up controllers for simulation. This won't work on real hardware -->
                 <plugin>mock_components/GenericSystem</plugin>
-              </xacro:if>
-              <xacro:if value="${use_gazebo}">
-                <plugin>gazebo_ros2_control/GazeboSystem</plugin>
-              </xacro:if>
-              <xacro:unless value="${use_mock_hardware or use_gazebo}">
-                <!-- Parameters to initialize the Components -->
-                <param name="families">${families}</param>
-                <param name="names">${names}</param>
-                <param name="hrdf_pkg">${hrdf_pkg}</param>
-                <param name="hrdf_file">${hrdf_file}</param>
-                <param name="gains_pkg">${gains_pkg}</param>
-                <param name="gains_file">${gains_file}</param>
-                <param name="home_position">${home_position}</param>
-                <plugin>hebi_hardware/HEBIHardwareInterface</plugin>
-              </xacro:unless>
             </hardware>
             <joint name="J1_base">
@@ -73,12 +49,4 @@
             </joint>
         </ros2_control>
-        <!-- Gazebo Classic plugins -->
-        <xacro:if value="${use_gazebo}">
-          <gazebo>
-            <plugin filename="libgazebo_ros2_control.so" name="gazebo_ros2_control">
-              <parameters>$(find hebi_a-2085-05_moveit_config)/config/ros2_controllers.yaml</parameters>
-            </plugin>
-          </gazebo>
-        </xacro:if>
     </xacro:macro>
 </robot>

File: hebi_a-2085-06-parallel-gripper_moveit_config/config/A-2085-06-parallel-gripper.ros2_control.xacro (robot description, xacro)
@@ -3,32 +3,8 @@
     <xacro:macro name="A-2085-06-parallel-gripper_ros2_control" params="name initial_positions_file">
         <xacro:property name="initial_positions" value="${load_yaml(initial_positions_file)['initial_positions']}"/>
-        <xacro:property name="home_position" value="${load_yaml(initial_positions_file)['home_position']}"/>
-        <xacro:property name="families" value="${load_yaml(initial_positions_file)['families']}"/>
-        <xacro:property name="names" value="${load_yaml(initial_positions_file)['names']}"/>
-        <xacro:property name="hrdf_pkg" value="${load_yaml(initial_positions_file)['hrdf_pkg']}"/>
-        <xacro:property name="hrdf_file" value="${load_yaml(initial_positions_file)['hrdf_file']}"/>
-        <xacro:property name="gains_pkg" value="${load_yaml(initial_positions_file)['gains_pkg']}"/>
-        <xacro:property name="gains_file" value="${load_yaml(initial_positions_file)['gains_file']}"/>
-        <xacro:property name="use_mock_hardware" value="${load_yaml(initial_positions_file)['use_mock_hardware']}"/>
-        <xacro:property name="use_gazebo" value="${load_yaml(initial_positions_file)['use_gazebo']}"/>
         <ros2_control name="${name}" type="system">
             <hardware>
-              <xacro:if value="${use_mock_hardware}">
+                <!-- By default, set up controllers for simulation. This won't work on real hardware -->
                 <plugin>mock_components/GenericSystem</plugin>
-              </xacro:if>
-              <xacro:if value="${use_gazebo}">
-                <plugin>gazebo_ros2_control/GazeboSystem</plugin>
-              </xacro:if>
-              <xacro:unless value="${use_mock_hardware or use_gazebo}">
-                <!-- Parameters to initialize the Components -->
-                <param name="families">${families}</param>
-                <param name="names">${names}</param>
-                <param name="hrdf_pkg">${hrdf_pkg}</param>
-                <param name="hrdf_file">${hrdf_file}</param>
-                <param name="gains_pkg">${gains_pkg}</param>
-                <param name="gains_file">${gains_file}</param>
-                <param name="home_position">${home_position}</param>
-                <plugin>hebi_hardware/HEBIHardwareInterface</plugin>
-              </xacro:unless>
             </hardware>
             <joint name="J1_base">

File: hebi_a-2085-06_moveit_config/config/A-2085-06.ros2_control.xacro (robot description, xacro)
@@ -3,32 +3,8 @@
     <xacro:macro name="A-2085-06_ros2_control" params="name initial_positions_file">
         <xacro:property name="initial_positions" value="${load_yaml(initial_positions_file)['initial_positions']}"/>
-        <xacro:property name="home_position" value="${load_yaml(initial_positions_file)['home_position']}"/>
-        <xacro:property name="families" value="${load_yaml(initial_positions_file)['families']}"/>
-        <xacro:property name="names" value="${load_yaml(initial_positions_file)['names']}"/>
-        <xacro:property name="hrdf_pkg" value="${load_yaml(initial_positions_file)['hrdf_pkg']}"/>
-        <xacro:property name="hrdf_file" value="${load_yaml(initial_positions_file)['hrdf_file']}"/>
-        <xacro:property name="gains_pkg" value="${load_yaml(initial_positions_file)['gains_pkg']}"/>
-        <xacro:property name="gains_file" value="${load_yaml(initial_positions_file)['gains_file']}"/>
-        <xacro:property name="use_mock_hardware" value="${load_yaml(initial_positions_file)['use_mock_hardware']}"/>
-        <xacro:property name="use_gazebo" value="${load_yaml(initial_positions_file)['use_gazebo']}"/>
         <ros2_control name="${name}" type="system">
             <hardware>
-              <xacro:if value="${use_mock_hardware}">
+                <!-- By default, set up controllers for simulation. This won't work on real hardware -->
                 <plugin>mock_components/GenericSystem</plugin>
-              </xacro:if>
-              <xacro:if value="${use_gazebo}">
-                <plugin>gazebo_ros2_control/GazeboSystem</plugin>
-              </xacro:if>
-              <xacro:unless value="${use_mock_hardware or use_gazebo}">
-                <!-- Parameters to initialize the Components -->
-                <param name="families">${families}</param>
-                <param name="names">${names}</param>
-                <param name="hrdf_pkg">${hrdf_pkg}</param>
-                <param name="hrdf_file">${hrdf_file}</param>
-                <param name="gains_pkg">${gains_pkg}</param>
-                <param name="gains_file">${gains_file}</param>
-                <param name="home_position">${home_position}</param>
-                <plugin>hebi_hardware/HEBIHardwareInterface</plugin>
-              </xacro:unless>
             </hardware>
             <joint name="J1_base">
@@ -81,12 +57,4 @@
             </joint>
         </ros2_control>
-        <!-- Gazebo Classic plugins -->
-        <xacro:if value="${use_gazebo}">
-          <gazebo>
-            <plugin filename="libgazebo_ros2_control.so" name="gazebo_ros2_control">
-              <parameters>$(find hebi_a-2085-06_moveit_config)/config/ros2_controllers.yaml</parameters>
-            </plugin>
-          </gazebo>
-        </xacro:if>
     </xacro:macro>
 </robot>
